File: noob_tester.sch (KiCad schematic (older format))
At the start: 30 parts, among them J1 Conn_01x10_Male, J2 Conn_01x10_Male, J3 Conn_01x10_Male, J4 Conn_01x10_Male, J5 Conn_01x10_Male, J6 Conn_01x10_Male, Q1 Q_NJFET_DGS, Q2 Q_NJFET_DGS, Q3 Q_NJFET_DGS, Q4 Q_NJFET_DGS

Commit message: swapped SOT-23 with SOT-723, generated gerber files
Parts:
- Q2, Q4: footprint Package_TO_SOT_SMD:SOT-23 -> Package_TO_SOT_SMD:SOT-723
Changed lines of the file:
@@
 F 0 "Q4" H 7441 2796 50  0000 L CNN
 F 1 "Q_NJFET_DGS" H 7441 2705 50  0000 L CNN
-F 2 "Package_TO_SOT_SMD:SOT-23" H 7450 2850 50  0001 C CNN
+F 2 "Package_TO_SOT_SMD:SOT-723" H 7450 2850 50  0001 C CNN
 F 3 "~" H 7250 2750 50  0001 C CNN
 	1    7250 2750
@@
 F 0 "Q2" H 6341 2796 50  0000 L CNN
 F 1 "Q_NJFET_DGS" H 6341 2705 50  0000 L CNN
-F 2 "Package_TO_SOT_SMD:SOT-23" H 6350 2850 50  0001 C CNN
+F 2 "Package_TO_SOT_SMD:SOT-723" H 6350 2850 50  0001 C CNN
 F 3 "~" H 6150 2750 50  0001 C CNN
 	1    6150 2750
-	1    0    0    -1
-$EndComp
-$Comp
-L power:GND #PWR0102
-U 1 1 5F3C22C8
-P 5700 3150
-F 0 "#PWR0102" H 5700 2900 50  0001 C CNN
-F 1 "GND" H 5705 2977 50  0000 C CNN
-F 2 "" H 5700 3150 50  0001 C CNN
-F 3 "" H 5700 3150 50  0001 C CNN
-	1    5700 3150
 	1    0    0    -1
 $EndComp
@@
 Wire Wire Line
 	3700 2200 3700 2300
+$Comp
+L power:GND #PWR0102
+U 1 1 5F3C22C8
+P 5700 3150
+F 0 "#PWR0102" H 5700 2900 50  0001 C CNN
+F 1 "GND" H 5705 2977 50  0000 C CNN
+F 2 "" H 5700 3150 50  0001 C CNN
+F 3 "" H 5700 3150 50  0001 C CNN
+	1    5700 3150
+	1    0    0    -1
+$EndComp
 $EndSCHEMATC
